File: hw/sch_pcb/USB_UART.kicad_sch (KiCad schematic)
At the start: 18 parts, among them J2 USBC_USB4105-GF-A, U5 USBLC6-2SC6, U6 FT231XQ

Commit message: Edit
Parts:
- added F?: Fuse, symbol Device:Fuse
- added J? (x2): SM06B-GHS-TB, Connector_JST:JST_GH_SM06B-GHS-TB_1x06-1MP_P1.25mm_Horizontal, symbol MLAB_CONNECTORS_JST:SM06B-GHS-TB
Connections:
- net +5V: now also J?.1, J?.1
- net GND: now also J?.6, J?.6, J?.MP, J?.MP
- net VBUS: now also F?.1; no longer C2.1, FB1.1
- net #CTS_USB renamed #CTS
- net #CTS: now also J?.5, J?.5
- net #RTS_USB renamed #RTS
- net #RTS: now also J?.4, J?.4
- net RXD_USB renamed RXD
- net RXD: now also J?.2, J?.3
- net TXD_USB renamed TXD
- net TXD: now also J?.2, J?.3
- new net: C2.1, F?.2, FB1.1
