File: hw/sch_pcb/TFUSBSERIAL01A.kicad_pcb (KiCad board)
At the start: 2 copper layers, 77.1 x 65 mm, 112 parts, among them J1 SM06B-GHS-TB, J2 USBC_USB4105-GF-A, J3 MCX 73415-1061, J4 MCX 73415-1061, Q3 BC817, Q4 BC817, Q5 BC817, U1 LM1117-3V3, U10 SPF5189Z, U2 Si1060-A-GM, U3 LSF0204, U4 LSF0204, U5 USBLC6-2SC6, U6 FT231XQ, U7 PE4259, U8 TPS22945DCKR, U9 PE4259, Y1 ABS07-120-32.768KHZ, Y2 ABM3B-30.000MHZ-10-1-U-T

Commit message: Edit
Parts:
- removed C10, C11, C9: 8,2pF, Capacitor_SMD:C_0603_1608Metric
- removed C12: 2.7pF, Capacitor_SMD:C_0603_1608Metric
- removed C13: 5.1pF, Capacitor_SMD:C_0603_1608Metric
- removed C14: 10nF, Capacitor_SMD:C_0603_1608Metric
- removed C15: 33pF, Capacitor_SMD:C_0603_1608Metric
- removed C16, C19, C22, C24, C25, C32, C35, C36: 100nF, Capacitor_SMD:C_0603_1608Metric
- removed C17, C30, C33: 100pF, Capacitor_SMD:C_0603_1608Metric
- removed C18, C20: 10uF, Capacitor_SMD:C_0805_2012Metric
- removed C21: NFM21PC105, Mlab_L:FIR_0805
- removed C23: 10uF, Capacitor_SMD:C_0603_1608Metric
- removed C26, C27, C31, C34: 1nF, Capacitor_SMD:C_0603_1608Metric
- removed C28, C29: 2p2, Capacitor_SMD:C_0603_1608Metric
- removed C6: 6.8pf, Capacitor_SMD:C_0603_1608Metric
- removed C7, C8: 15pF, Capacitor_SMD:C_0603_1608Metric
- removed D4: GREEN, LED_SMD:LED_0603_1608Metric_Castellated
- removed D5: RED, LED_SMD:LED_0603_1608Metric_Castellated
- removed D6, D7: 15MQ040N, Diode_SMD:D_SMA
- removed FL1: SAW_AFS434S3-T_AFS869S3-T, MLAB_SAW:ABRACON_AFS
- removed J4: MCX 73415-1061, Mlab_CON:MCX_Molex_73415-1061
- removed L1, L2: 0R, Inductor_SMD:L_0805_2012Metric
- removed L10, L9: 56nH, Inductor_SMD:L_0805_2012Metric
- removed L11, L12, L16: 100nH, Inductor_SMD:L_0805_2012Metric
- removed L13: 6n8, Inductor_SMD:L_0805_2012Metric
- removed L14: 74279204, Inductor_SMD:L_0805_2012Metric
- removed L15: 1n5H, Inductor_SMD:L_0805_2012Metric
- removed L3, L4, L5, L6: 18nH, Inductor_SMD:L_0805_2012Metric
- removed L7: 39nH, Inductor_SMD:L_0805_2012Metric
- removed L8: 220nH, Inductor_SMD:L_0805_2012Metric
- removed Q3, Q4, Q5: BC817, Package_TO_SOT_SMD:SOT-23
- removed R10, R26, R29, R7, R9: 10k, Resistor_SMD:R_0603_1608Metric
- removed R11, R12: 200kR, Resistor_SMD:R_0603_1608Metric
- removed R13, R14, R15, R16, R17, R18, R19, R20, R24, R8: 1k, Resistor_SMD:R_0603_1608Metric
- removed R21: 0R, Resistor_SMD:R_0603_1608Metric
- removed R22, R23: 150R, Resistor_SMD:R_0603_1608Metric
- removed R25: 4k7, Resistor_SMD:R_0603_1608Metric
- removed R27, R28: 270R, Resistor_SMD:R_0603_1608Metric
- removed R30: 330R, Resistor_SMD:R_0603_1608Metric
- removed R31, R32: 5k1, Resistor_SMD:R_0603_1608Metric
- removed U10: SPF5189Z, Package_TO_SOT_SMD:SOT-89-3
- removed U3, U4: LSF0204, Package_SO:TSSOP-14_4.4x5mm_P0.65mm
- removed U5: USBLC6-2SC6, Package_TO_SOT_SMD:SOT-23-6
- removed U6: FT231XQ, Package_DFN_QFN:QFN-20-1EP_4x4mm_P0.5mm_EP2.5x2.5mm
- removed U7, U9: PE4259, Package_TO_SOT_SMD:SOT-363_SC-70-6
- removed U8: TPS22945DCKR, Package_TO_SOT_SMD:SOT-353_SC-70-5
- removed Y1: ABS07-120-32.768KHZ, Mlab_XTAL:ABS07
- removed Y2: ABM3B-30.000MHZ-10-1-U-T, Crystal:Crystal_SMD_Abracon_ABM3B-4Pin_5.0x3.2mm
- added F1: Fuse, Mlab_F:1812, B.Cu at (6.19, -7.14)
- C1: value 10uF -> 10nF; footprint Capacitor_SMD:C_0805_2012Metric -> Capacitor_SMD:C_0603_1608Metric
- C2: value 10nF -> 100nF
- C3: footprint Capacitor_SMD:C_0805_2012Metric -> Capacitor_SMD:C_0603_1608Metric
- C4: value 6.8pf -> 100nF
- C5: value 10uF -> 100nF; footprint Capacitor_SMD:C_0805_2012Metric -> Capacitor_SMD:C_0603_1608Metric
- D1: value RED -> 15MQ040N; footprint LED_SMD:LED_0603_1608Metric_Castellated -> Diode_SMD:D_SMA
- J1: value SM06B-GHS-TB -> USBC_USB4105-GF-A; footprint Connector_JST:JST_GH_SM06B-GHS-TB_1x06-1MP_P1.25mm_Horizontal -> Mlab_CON:USBC GCT_USB4105-GF-A
- J2: value USBC_USB4105-GF-A -> SM06B-GHS-TB; footprint Mlab_CON:USBC GCT_USB4105-GF-A -> Connector_JST:JST_GH_SM06B-GHS-TB_1x06-1MP_P1.25mm_Horizontal
- J3: value MCX 73415-1061 -> SM06B-GHS-TB; footprint Mlab_CON:MCX_Molex_73415-1061 -> Connector_JST:JST_GH_SM06B-GHS-TB_1x06-1MP_P1.25mm_Horizontal
- R1: value 0R -> 5k1
- R2: value 1k5 -> 5k1
- R3: value 1k5 -> 4k7
- R4: value 1k5 -> 10k
- R5: value 1k5 -> 270R
- R6: value 1k -> 270R
- U1: value LM1117-3V3 -> USBLC6-2SC6; footprint Mlab_IO:SOT-223 -> Package_TO_SOT_SMD:SOT-23-6
- U2: value Si1060-A-GM -> FT231XQ; footprint Package_DFN_QFN:QFN-36-1EP_5x6mm_P0.5mm_EP3.6x4.1mm_ThermalVias -> Package_DFN_QFN:QFN-20-1EP_4x4mm_P0.5mm_EP2.5x2.5mm
- moved R3 53.7 mm to (-18.0, -14.9)
- moved R4 53.0 mm to (-13.3, -14.5)
- moved C3 46.1 mm to (13.3, -2.48), turned to -90 degrees
- moved D1 45.1 mm to (16.8, -4.03), turned to -90 degrees
- moved C2 43.2 mm to (18.3, -18.9), turned to 180 degrees
- moved C1 42.7 mm to (7.54, -2.48), turned to -90 degrees
- moved J3 41.1 mm to (26.8, -7.50), turned to -90 degrees
- moved C5 40.0 mm to (16.8, -10.8), turned to 0 degrees
- moved FB1 38.1 mm to (10.5, -4.45)
- moved R5 34.2 mm to (3.47, -27.4)
- moved U1 30.1 mm to (13.6, -15.0), turned to 180 degrees
- moved R2 29.2 mm to (11.0, -21.1), turned to 0 degrees
- moved J2 28.1 mm to (26.8, -22.5), turned to -90 degrees
- moved D3 27.9 mm to (4.12, -24.9), turned to 0 degrees
- moved D2 25.8 mm to (7.59, -23.8), turned to 0 degrees
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Connections:
- C1 pad 1: +5V -> Net-(C1-Pad1)
- C2 pad 1: /USB UART/VBUS -> Net-(C2-Pad1)
- C3 pad 1: +3V3 -> Net-(C3-Pad1)
- C4 pad 1: Net-(C4-Pad1) -> Net-(C3-Pad1)
- C5 pad 1: +3V3 -> GND
- C5 pad 2: GND -> Net-(C2-Pad1)
- D1 pad 1: Net-(D1-Pad1) -> +5V
- D1 pad 2: +5V -> Net-(C3-Pad1)
- D2 pad 2: /P1.4 -> +5V
- D3 pad 2: /P1.5 -> +5V
- FB1 pad 1: /USB UART/VBUS -> Net-(C1-Pad1)
- FB1 pad 2: Net-(C23-Pad1) -> Net-(C3-Pad1)
- J3 pad 1: /RFSWITCH/RX/TX_1 -> +5V
- J3 pad 2: GND -> /RXD
- R1 pad 1: +3V3 -> Net-(J1-PadA5)
- R1 pad 2: Net-(L8-Pad1) -> GND
- R2 pad 1: +5V -> Net-(J1-PadB5)
- R2 pad 2: RX -> GND
- R3 pad 1: +5V -> Net-(C3-Pad1)
- R3 pad 2: TX -> Net-(R3-Pad2)
- R4 pad 1: +5V -> Net-(R3-Pad2)
- R4 pad 2: RTS_SI -> GND
- R5 pad 1: +5V -> Net-(D2-Pad1)
- R5 pad 2: CTS_SI -> /RXLED/CBUS1
- R6 pad 1: USB_ON -> Net-(D3-Pad1)
- R6 pad 2: Net-(Q3-Pad1) -> /TXLED/CBUS2
- U1 pad 1: GND -> /DM
- U1 pad 2: +3V3 -> GND
- U1 pad 3: +5V -> /DP
- U1 pad 4: +3V3 -> /D+
- U2 pad 1: unconnected-(U2-Pad1) -> /RXD
- U2 pad 10: unconnected-(U2-Pad10) -> Net-(C2-Pad1)
- U2 pad 11: GPIO3 -> Net-(R3-Pad2)
- U2 pad 12: Net-(C13-Pad1) -> Net-(C3-Pad1)
- U2 pad 13: Net-(C12-Pad1) -> GND
- U2 pad 14: GND -> /RXLED/CBUS1
- U2 pad 15: GND -> unconnected-(U2-Pad15)
- U2 pad 16: Net-(C11-Pad1) -> unconnected-(U2-Pad16)
- U2 pad 17: GND -> /TXD
- U2 pad 18: Net-(C15-Pad1) -> unconnected-(U2-Pad18)
- U2 pad 19: unconnected-(U2-Pad19) -> /#RTS
- U2 pad 2: Net-(U2-Pad2) -> unconnected-(U2-Pad2)
- U2 pad 20: Net-(C15-Pad1) -> Net-(C2-Pad1)
- U2 pad 21: unconnected-(U2-Pad21) -> GND
- U2 pad 3: Net-(U2-Pad3) -> GND
- U2 pad 5: /P1.5 -> unconnected-(U2-Pad5)
- U2 pad 6: /P1.4 -> /#CTS
- U2 pad 7: Net-(U2-Pad7) -> /TXLED/CBUS2
- U2 pad 8: Net-(U2-Pad8) -> /DP
- U2 pad 9: GND -> /DM
Routing:
- net /D-: track 0.00 -> 9.01 mm
- net /D+: track 0.00 -> 6.53 mm, vias 0 -> 2
Other:
- board size 77.1 x 65 mm -> 30 x 30 mm

Commit message: Edit PCB
Parts:
- added M1: HOLE_TF, Mlab_Mechanical:dira_3mm, F.Cu at (2.92, -0.13)
- added M2: HOLE_TF, Mlab_Mechanical:dira_3mm, F.Cu at (20.6, 0.25)
- added M3: HOLE_TF, Mlab_Mechanical:dira_3mm, F.Cu at (3.30, -29.8)
- added M4: HOLE_TF, Mlab_Mechanical:dira_3mm, F.Cu at (11.4, 0.00)
- added M5: HOLE_TF, Mlab_Mechanical:dira_3mm, F.Cu at (24.4, -29.8)
- added M6: HOLE_TF, Mlab_Mechanical:dira_3mm, F.Cu at (15.2, -30.0)
- moved R3 37.7 mm to (18.9, -22.5), turned to 180 degrees
- moved R4 30.0 mm to (15.6, -22.5), turned to 180 degrees
- moved R5 9.46 mm to (11.8, -22.9), turned to -90 degrees
- moved R1 7.97 mm to (4.19, -22.9), turned to 90 degrees
- moved C4 6.78 mm to (19.8, -19.6), turned to 0 degrees
- moved R2 4.99 mm to (6.35, -22.9), turned to 90 degrees
- moved C5 4.97 mm to (21.7, -10.7), turned to 90 degrees
- moved C3 4.66 mm to (13.9, -7.11), turned to 0 degrees
- moved C1 4.06 mm to (11.5, -3.17), turned to 0 degrees
- moved D2 3.23 mm to (8.00, -27.0), turned to 90 degrees
- moved R6 2.64 mm to (9.14, -22.9), turned to -90 degrees
- moved C2 2.53 mm to (15.8, -19.1)
- moved D3 2.29 mm to (5.00, -27.0), turned to 90 degrees
- moved F1 2.18 mm to (7.11, -5.16), turned to -90 degrees
- moved D1 1.76 mm to (18.4, -4.70)
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Routing:
- net /#CTS: track 0.00 -> 37.1 mm, vias 0 -> 2
- net /RXD: track 0.00 -> 25.5 mm, vias 0 -> 3
- net /TXD: track 0.00 -> 24.1 mm, vias 0 -> 2
- net /#RTS: track 0.00 -> 20.9 mm
- net /VBUS: track 0.00 -> 19.4 mm, vias 0 -> 3
- net Net-(C3-Pad1): track 0.00 -> 16.3 mm
- net /TXLED/CBUS2: track 0.00 -> 12.5 mm, vias 0 -> 2
- net /RXLED/CBUS1: track 0.00 -> 11.8 mm, vias 0 -> 2
- net Net-(J1-PadA5): track 0.00 -> 11.2 mm
- net Net-(J1-PadB5): track 0.00 -> 7.78 mm
- net Net-(R3-Pad2): track 0.00 -> 7.30 mm
- net Net-(C1-Pad1): track 0.00 -> 5.55 mm
- net Net-(D3-Pad1): track 0.00 -> 5.15 mm
- net Net-(D2-Pad1): track 0.00 -> 4.82 mm
- net /DP: track 0.00 -> 3.03 mm
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
Commit message: EDIT PCB
Parts:
- moved M6 2.74 mm to (12.5, -30.0)
- moved M2 1.94 mm to (22.5, 0.00)
- moved M5 1.89 mm to (22.5, -30.0)
- moved M4 1.07 mm to (12.5, 0.00)
- moved M3 0.82 mm to (2.50, -30.0)
- moved C2 0.80 mm to (15.0, -18.9)
- moved M1 0.44 mm to (2.50, 0.00)
Connections:
- C4 pad 1: Net-(C3-Pad1) -> +5V
- R3 pad 1: Net-(C3-Pad1) -> +5V
- U2 pad 12: Net-(C3-Pad1) -> +5V
Routing:
- net +5V: track 0.00 -> 65.4 mm, vias 0 -> 4
- net Net-(C2-Pad1): track 0.00 -> 14.2 mm, vias 0 -> 2
- net GND: track 0.00 -> 11.9 mm, vias 0 -> 50
- net Net-(C3-Pad1): track 16.3 -> 10.3 mm
- net /#CTS: track 37.1 -> 40.5 mm
- net /RXD: track 25.5 -> 26.5 mm
- net /#RTS: track 20.9 -> 20.2 mm
- added copper zone on B.Cu, net GND
- added copper zone on F.Cu, net GND

Commit message: Edit PCB
Parts:
- added G***: LOGO, MLAB_LOGA:TF, F.Cu at (12.4, -3.94)
Other:
- board text added: "2021"
- board text added: "TFUSBSERIAL01A"
- board text added: "to DEVICE"
- board text added: "to FMU"

Commit message: Edit SCH and PCB
Parts:
- moved G*** 0.40 mm to (12.1, -3.81)
Connections:
- J2 pad 4: /#RTS -> /#CTS
- J2 pad 5: /#CTS -> /#RTS
Routing:
- net /#CTS: track 40.5 -> 42.1 mm
- net /#RTS: track 20.2 -> 19.2 mm

Commit message: Edit PCB
Parts:
- removed G***: LOGO, MLAB_LOGA:TF
- added D4: GREEN, LED_SMD:LED_0603_1608Metric, B.Cu at (13.5, -9.65)
- added R7: 270R, Resistor_SMD:R_0603_1608Metric, B.Cu at (39.6, -15.2)
- D2, D3: footprint LED_SMD:LED_0603_1608Metric_Castellated -> LED_SMD:LED_0603_1608Metric
- F1: value Fuse -> 750mA
- moved R3 3.18 mm to (16.0, -21.1), turned to 0 degrees
- moved R4 0.77 mm to (16.0, -23.1)
Connections:
- R3 pad 1: +5V -> /VBUS
Routing:
- net /VBUS: track 19.4 -> 25.7 mm
- net GND: track 11.9 -> 10.8 mm, vias 50 -> 49
- net /#CTS: track 42.1 -> 41.5 mm
- net Net-(U2-~{RESET}): track 7.30 -> 6.79 mm
Other:
- board text added: "2023"
- board text added: "as FMU"
- board text removed: "2021"
- board text removed: "to DEVICE"
