File: hw/sch_pcb/TFUSBSERIAL01A.kicad_sch (KiCad schematic)
At the start: 41 parts, among them U1 LM1117-3V3, U2 Si1060-A-GM, Y1 ABS07-120-32.768KHZ, Y2 ABM3B-30.000MHZ-10-1-U-T

Commit message: Edit
Parts:
- removed C1, C18, C20, C3, C5: 10uF, Capacitor_SMD:C_0805_2012Metric, symbol Device:C_Small
- removed C10, C11, C9: 8,2pF, Capacitor_SMD:C_0603_1608Metric, symbol Device:C_Small
- removed C12: 2.7pF, Capacitor_SMD:C_0603_1608Metric, symbol Device:C_Small
- removed C13: 5.1pF, Capacitor_SMD:C_0603_1608Metric, symbol Device:C_Small
- removed C14: 10nF, Capacitor_SMD:C_0603_1608Metric, symbol Device:C_Small
- removed C15: 33pF, Capacitor_SMD:C_0603_1608Metric, symbol Device:C_Small
- removed C16, C19: 100nF, Capacitor_SMD:C_0603_1608Metric, symbol Device:C_Small
- removed C17: 100pF, Capacitor_SMD:C_0603_1608Metric, symbol Device:C_Small
- removed C21: NFM21PC105, Mlab_L:FIR_0805, symbol Device:Filter_EMI_C
- removed C4, C6: 6.8pf, Capacitor_SMD:C_0603_1608Metric, symbol Device:C_Small
- removed C7, C8: 15pF, Capacitor_SMD:C_0603_1608Metric, symbol Device:C_Small
- removed L1, L2: 0R, Inductor_SMD:L_0805_2012Metric, symbol Device:L_Small
- removed L10, L9: 56nH, Inductor_SMD:L_0805_2012Metric, symbol Device:L_Small
- removed L3, L4, L5, L6: 18nH, Inductor_SMD:L_0805_2012Metric, symbol Device:L_Small
- removed L7: 39nH, Inductor_SMD:L_0805_2012Metric, symbol Device:L_Small
- removed L8: 220nH, Inductor_SMD:L_0805_2012Metric, symbol Device:L_Small
- removed R20: 1k, Resistor_SMD:R_0603_1608Metric, symbol Device:R
- removed R21: 0R, Resistor_SMD:R_0603_1608Metric, symbol Device:R
- removed R22, R23: 150R, Resistor_SMD:R_0603_1608Metric, symbol Device:R
- removed U1: LM1117-3V3, Mlab_IO:SOT-223, symbol MLAB_U:LM1117
- removed U2: Si1060-A-GM, Package_DFN_QFN:QFN-36-1EP_5x6mm_P0.5mm_EP3.6x4.1mm_ThermalVias, symbol MLAB_IO:Si1060-A-GM
- removed Y1: ABS07-120-32.768KHZ, Mlab_XTAL:ABS07, symbol Device:Crystal
- removed Y2: ABM3B-30.000MHZ-10-1-U-T, Crystal:Crystal_SMD_Abracon_ABM3B-4Pin_5.0x3.2mm, symbol Device:Crystal_GND24
- added C1: 10nF, Capacitor_SMD:C_0603_1608Metric, symbol Device:C
- added C2, C4, C5: 100nF, Capacitor_SMD:C_0603_1608Metric, symbol Device:C
- added C3: 10uF, Capacitor_SMD:C_0603_1608Metric, symbol Device:C
- added D1: 15MQ040N, Diode_SMD:D_SMA, symbol Device:D
- added F1: Fuse, Mlab_F:1812, symbol Device:Fuse
- added FB1: BLM21PG300SN1D, Inductor_SMD:L_0805_2012Metric, symbol Device:FerriteBead_Small
- added J1: USBC_USB4105-GF-A, Mlab_CON:USBC GCT_USB4105-GF-A, symbol MLAB_CONNECTORS:USBC_USB4105-GF-A
- added J2, J3: SM06B-GHS-TB, Connector_JST:JST_GH_SM06B-GHS-TB_1x06-1MP_P1.25mm_Horizontal, symbol MLAB_CONNECTORS_JST:SM06B-GHS-TB
- added R2: 5k1, Resistor_SMD:R_0603_1608Metric, symbol Device:R
- added R3: 4k7, Resistor_SMD:R_0603_1608Metric, symbol Device:R
- added R4: 10k, Resistor_SMD:R_0603_1608Metric, symbol Device:R
- added R5, R6: 270R, Resistor_SMD:R_0603_1608Metric, symbol Device:R
- added U1: USBLC6-2SC6, Package_TO_SOT_SMD:SOT-23-6, symbol Power_Protection:USBLC6-2SC6
- added U2: FT231XQ, Package_DFN_QFN:QFN-20-1EP_4x4mm_P0.5mm_EP2.5x2.5mm, symbol Interface_USB:FT231XQ
- R1: value 0R -> 5k1; UST_ID 5c70984512875079b91f896b -> 5fa0fc3e12875025b3977997
Connections:
- net P1.4 is gone; now on net +5V: D2.2 (A)
- net P1.5 is gone; now on net +5V: D3.2 (A)
- net +5V: now also D1.1 (K), J2.1, J3.1
- net GND: now also R1.2, C1.2, C2.2, C3.2, C4.2, C5.1, J1.A1/B12 (GND), J1.B1/A12 (GND), J1.G1 (SHIELD), J1.G2 (SHIELD), J1.G3 (SHIELD), J1.G4 (SHIELD), J2.6, J2.MP, J3.6, J3.MP, R2.2, R4.2, U1.2 (GND), U2.13 (GND), U2.21 (GND), U2.3 (GND)
- net at D2.1 (K): now also R5.1
- net at D3.1 (K): now also R6.1
- net +3V3: no longer names the net of R1.1
- net +3V3: now also J1.A5 (CC1)
- new net: R3.2, R4.1, U2.11 (~RESET)
- new net: J1.B5 (CC2), R2.1
- new net: C2.1, C5.2, U2.10 (3V3OUT), U2.20 (VCCIO)
- new net: C1.1, F1.2, FB1.1
- new net: C3.1, C4.1, D1.2 (A), FB1.2, R3.1, U2.12 (VCC)
- new net #CTS: J2.5, J3.5, U2.6 (~CTS)
- new net #RTS: J2.4, J3.4, U2.19 (~RTS)
- new net D+: J1.A6 (D+), J1.B6 (D+), U1.4 (I/O2)
- new net D-: J1.A7 (D-), J1.B7 (D-), U1.6 (I/O1)
- new net DM: U1.1 (I/O1), U2.9 (USBDM)
- new net DP: U1.3 (I/O2), U2.8 (USBDP)
- new net RXD: J2.3, J3.2, U2.1 (RXD)
- new net RXLED/CBUS1: R5.2, U2.14 (CBUS1)
- new net TXD: J2.2, J3.3, U2.17 (TXD)
- new net TXLED/CBUS2: R6.2, U2.7 (CBUS2)
- new net VBUS: F1.1, J1.A4/B9 (VBUS), J1.B4/A9 (VBUS), U1.5 (VBUS)
- no-connect marks 7 -> 8
Other:
- removed sheet RFSWITCH
- removed sheet UART SWITCH
- removed sheet USB UART
- note added: "Budou tu LED?"
- note removed: "433MHz"

Commit message: Edit PCB
Parts:
- added M1, M2, M3, M4, M5, M6: HOLE_TF, Mlab_Mechanical:dira_3mm, symbol MLAB_MECHANICAL:HOLE_TF
Changed lines of the file:
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@@
     (effects (font (size 1.27 1.27)) (justify right bottom))
+  )
+  (symbol (lib_id "MLAB_MECHANICAL:HOLE_TF") (at 197.485 15.24 0) (unit 1)
+    (in_bom yes) (on_board yes) (fields_autoplaced)
+    (property "Reference" "M1" (id 0) (at 198.8821 14.3524 0)
+      (effects (font (size 1.524 1.524)) (justify left))
+    )
+    (property "Value" "HOLE_TF" (id 1) (at 198.8821 17.06 0)
+      (effects (font (size 1.524 1.524)) (justify left))
+    )
+    (property "Footprint" "Mlab_Mechanical:dira_3mm" (id 2) (at 197.485 15.24 0)
+      (effects (font (size 1.524 1.524)) hide)
+    )
+    (property "Datasheet" "" (id 3) (at 197.485 15.24 0)
+      (effects (font (size 1.524 1.524)))
+    )
+  )
+  (symbol (lib_id "MLAB_MECHANICAL:HOLE_TF") (at 197.485 21.59 0) (unit 1)
+    (in_bom yes) (on_board yes) (fields_autoplaced)
+    (property "Reference" "M2" (id 0) (at 198.8821 20.7024 0)
+      (effects (font (size 1.524 1.524)) (justify left))
+    )
+    (property "Value" "HOLE_TF" (id 1) (at 198.8821 23.41 0)
+      (effects (font (size 1.524 1.524)) (justify left))
+    )
+    (property "Footprint" "Mlab_Mechanical:dira_3mm" (id 2) (at 197.485 21.59 0)
+      (effects (font (size 1.524 1.524)) hide)
+    )
+    (property "Datasheet" "" (id 3) (at 197.485 21.59 0)
+      (effects (font (size 1.524 1.524)))
+    )
+  )
+  (symbol (lib_id "MLAB_MECHANICAL:HOLE_TF") (at 211.455 15.24 0) (unit 1)
+    (in_bom yes) (on_board yes) (fields_autoplaced)
+    (property "Reference" "M3" (id 0) (at 212.8521 14.3524 0)
+      (effects (font (size 1.524 1.524)) (justify left))
+    )
+    (property "Value" "HOLE_TF" (id 1) (at 212.8521 17.06 0)
+      (effects (font (size 1.524 1.524)) (justify left))
+    )
+    (property "Footprint" "Mlab_Mechanical:dira_3mm" (id 2) (at 211.455 15.24 0)
+      (effects (font (size 1.524 1.524)) hide)
+    )
+    (property "Datasheet" "" (id 3) (at 211.455 15.24 0)
+      (effects (font (size 1.524 1.524)))
+    )
+  )
+  (symbol (lib_id "MLAB_MECHANICAL:HOLE_TF") (at 211.455 21.59 0) (unit 1)
+    (in_bom yes) (on_board yes) (fields_autoplaced)
+    (property "Reference" "M4" (id 0) (at 212.8521 20.7024 0)
+      (effects (font (size 1.524 1.524)) (justify left))
+    )
+    (property "Value" "HOLE_TF" (id 1) (at 212.8521 23.41 0)
+      (effects (font (size 1.524 1.524)) (justify left))
+    )
+    (property "Footprint" "Mlab_Mechanical:dira_3mm" (id 2) (at 211.455 21.59 0)
+      (effects (font (size 1.524 1.524)) hide)
+    )
+    (property "Datasheet" "" (id 3) (at 211.455 21.59 0)
+      (effects (font (size 1.524 1.524)))
+    )
+  )
+  (symbol (lib_id "MLAB_MECHANICAL:HOLE_TF") (at 224.155 15.24 0) (unit 1)
+    (in_bom yes) (on_board yes) (fields_autoplaced)
+    (property "Reference" "M5" (id 0) (at 225.5521 14.3524 0)
+      (effects (font (size 1.524 1.524)) (justify left))
+    )
+    (property "Value" "HOLE_TF" (id 1) (at 225.5521 17.06 0)
+      (effects (font (size 1.524 1.524)) (justify left))
+    )
+    (property "Footprint" "Mlab_Mechanical:dira_3mm" (id 2) (at 224.155 15.24 0)
+      (effects (font (size 1.524 1.524)) hide)
+    )
+    (property "Datasheet" "" (id 3) (at 224.155 15.24 0)
+      (effects (font (size 1.524 1.524)))
+    )
+  )
+  (symbol (lib_id "MLAB_MECHANICAL:HOLE_TF") (at 224.155 21.59 0) (unit 1)
+    (in_bom yes) (on_board yes) (fields_autoplaced)
+    (property "Reference" "M6" (id 0) (at 225.5521 20.7024 0)
+      (effects (font (size 1.524 1.524)) (justify left))
+    )
+    (property "Value" "HOLE_TF" (id 1) (at 225.5521 23.41 0)
+      (effects (font (size 1.524 1.524)) (justify left))
+    )
+    (property "Footprint" "Mlab_Mechanical:dira_3mm" (id 2) (at 224.155 21.59 0)
+      (effects (font (size 1.524 1.524)) hide)
+    )
+    (property "Datasheet" "" (id 3) (at 224.155 21.59 0)
+      (effects (font (size 1.524 1.524)))
+    )
   )
   (symbol (lib_id "power:+5V") (at 138.43 53.975 0) (unit 1)
@@
       (reference "J3") (unit 1) (value "SM06B-GHS-TB") (footprint "Connector_JST:JST_GH_SM06B-GHS-TB_1x06-1MP_P1.25mm_Horizontal")
     )
+    (path "/07150fcc-da73-41e8-b5bc-83b21169905a"
+      (reference "M1") (unit 1) (value "HOLE_TF") (footprint "Mlab_Mechanical:dira_3mm")
+    )
+    (path "/b96fd542-3f19-4d43-96de-688022c1a9e1"
+      (reference "M2") (unit 1) (value "HOLE_TF") (footprint "Mlab_Mechanical:dira_3mm")
+    )
+    (path "/3b04b616-4d75-42e2-90fd-a67aacee2528"
+      (reference "M3") (unit 1) (value "HOLE_TF") (footprint "Mlab_Mechanical:dira_3mm")
+    )
+    (path "/74f42d80-c53a-4cd1-81c3-1ca032ef4173"
+      (reference "M4") (unit 1) (value "HOLE_TF") (footprint "Mlab_Mechanical:dira_3mm")
+    )
+    (path "/daf55a08-03f8-4aac-ab5b-3c300be303fe"
+      (reference "M5") (unit 1) (value "HOLE_TF") (footprint "Mlab_Mechanical:dira_3mm")
+    )
+    (path "/ad796685-f59e-4e5d-b6b6-55644de7de0b"
+      (reference "M6") (unit 1) (value "HOLE_TF") (footprint "Mlab_Mechanical:dira_3mm")
+    )
     (path "/554d742a-fd71-4249-ab41-03042967f073"

Commit message: EDIT PCB
Connections:
- net +5V: now also C4.1, R3.1, U2.12 (VCC)
- net at C3.1, D1.2 (A), FB1.2: no longer C4.1, R3.1, U2.12 (VCC)
Other:
- moved on the sheet: C4, D1
Changed lines of the file:
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@@
   (junction (at 95.25 109.22) (diameter 1.016) (color 0 0 0 0))
   (junction (at 106.68 93.98) (diameter 1.016) (color 0 0 0 0))
-  (junction (at 109.22 66.04) (diameter 1.016) (color 0 0 0 0))
   (junction (at 114.3 66.04) (diameter 1.016) (color 0 0 0 0))
-  (junction (at 125.73 66.04) (diameter 1.016) (color 0 0 0 0))
+  (junction (at 128.905 66.04) (diameter 1.016) (color 0 0 0 0))
   (junction (at 138.43 66.04) (diameter 1.016) (color 0 0 0 0))
   (junction (at 140.97 133.35) (diameter 1.016) (color 0 0 0 0))
@@
     (stroke (width 0) (type solid) (color 0 0 0 0))
   )
-  (wire (pts (xy 95.25 80.01) (xy 95.25 99.06))
+  (wire (pts (xy 95.25 94.615) (xy 95.25 99.06))
     (stroke (width 0) (type solid) (color 0 0 0 0))
   )
@@
     (stroke (width 0) (type solid) (color 0 0 0 0))
   )
-  (wire (pts (xy 105.41 66.04) (xy 109.22 66.04))
+  (wire (pts (xy 105.41 66.04) (xy 114.3 66.04))
     (stroke (width 0) (type solid) (color 0 0 0 0))
   )
@@
     (stroke (width 0) (type solid) (color 0 0 0 0))
   )
-  (wire (pts (xy 109.22 66.04) (xy 109.22 80.01))
-    (stroke (width 0) (type solid) (color 0 0 0 0))
-  )
-  (wire (pts (xy 109.22 66.04) (xy 114.3 66.04))
-    (stroke (width 0) (type solid) (color 0 0 0 0))
-  )
-  (wire (pts (xy 109.22 80.01) (xy 95.25 80.01))
-    (stroke (width 0) (type solid) (color 0 0 0 0))
-  )
   (wire (pts (xy 114.3 66.04) (xy 114.3 67.31))
     (stroke (width 0) (type solid) (color 0 0 0 0))
   )
-  (wire (pts (xy 114.3 66.04) (xy 125.73 66.04))
+  (wire (pts (xy 114.3 66.04) (xy 118.11 66.04))
     (stroke (width 0) (type solid) (color 0 0 0 0))
   )
@@
     (stroke (width 0) (type solid) (color 0 0 0 0))
   )
-  (wire (pts (xy 125.73 66.04) (xy 125.73 67.31))
-    (stroke (width 0) (type solid) (color 0 0 0 0))
-  )
-  (wire (pts (xy 125.73 66.04) (xy 138.43 66.04))
-    (stroke (width 0) (type solid) (color 0 0 0 0))
-  )
-  (wire (pts (xy 125.73 74.93) (xy 125.73 76.2))
-    (stroke (width 0) (type solid) (color 0 0 0 0))
-  )
-  (wire (pts (xy 138.43 53.975) (xy 138.43 55.245))
-    (stroke (width 0) (type solid) (color 0 0 0 0))
-  )
-  (wire (pts (xy 138.43 62.865) (xy 138.43 66.04))
+  (wire (pts (xy 125.73 66.04) (xy 128.905 66.04))
+    (stroke (width 0) (type solid) (color 0 0 0 0))
+  )
+  (wire (pts (xy 128.905 66.04) (xy 128.905 67.31))
+    (stroke (width 0) (type solid) (color 0 0 0 0))
+  )
+  (wire (pts (xy 128.905 66.04) (xy 138.43 66.04))
+    (stroke (width 0) (type solid) (color 0 0 0 0))
+  )
+  (wire (pts (xy 128.905 74.93) (xy 128.905 76.2))
+    (stroke (width 0) (type solid) (color 0 0 0 0))
+  )
+  (wire (pts (xy 138.43 53.975) (xy 138.43 66.04))
     (stroke (width 0) (type solid) (color 0 0 0 0))
   )
@@
     )
   )
+  (symbol (lib_id "power:+5V") (at 95.25 94.615 0) (unit 1)
+    (in_bom yes) (on_board yes) (fields_autoplaced)
+    (property "Reference" "#PWR?" (id 0) (at 95.25 98.425 0)
+      (effects (font (size 1.27 1.27)) hide)
+    )
+    (property "Value" "+5V" (id 1) (at 95.25 91.0676 0))
+    (property "Footprint" "" (id 2) (at 95.25 94.615 0)
+      (effects (font (size 1.27 1.27)) hide)
+    )
+    (property "Datasheet" "" (id 3) (at 95.25 94.615 0)
+      (effects (font (size 1.27 1.27)) hide)
+    )
+    (pin "1")
+  )
   (symbol (lib_id "power:+5V") (at 138.43 53.975 0) (unit 1)
     (in_bom yes) (on_board yes) (fields_autoplaced)
@@
     (pin "1")
   )
-  (symbol (lib_id "power:GND") (at 125.73 76.2 0) (unit 1)
-    (in_bom yes) (on_board yes)
-    (property "Reference" "#PWR0113" (id 0) (at 125.73 82.55 0)
-      (effects (font (size 1.27 1.27)) hide)
-    )
-    (property "Value" "GND" (id 1) (at 125.8443 80.5244 0))
-    (property "Footprint" "" (id 2) (at 125.73 76.2 0)
-      (effects (font (size 1.27 1.27)) hide)
-    )
-    (property "Datasheet" "" (id 3) (at 125.73 76.2 0)
+  (symbol (lib_id "power:GND") (at 128.905 76.2 0) (unit 1)
+    (in_bom yes) (on_board yes)
+    (property "Reference" "#PWR0113" (id 0) (at 128.905 82.55 0)
+      (effects (font (size 1.27 1.27)) hide)
+    )
+    (property "Value" "GND" (id 1) (at 129.0193 80.5244 0))
+    (property "Footprint" "" (id 2) (at 128.905 76.2 0)
+      (effects (font (size 1.27 1.27)) hide)
+    )
+    (property "Datasheet" "" (id 3) (at 128.905 76.2 0)
       (effects (font (size 1.27 1.27)) hide)
     )
@@
     (pin "2")
   )
-  (symbol (lib_id "Device:D") (at 138.43 59.055 270) (unit 1)
-    (in_bom yes) (on_board yes) (fields_autoplaced)
-    (property "Reference" "D1" (id 0) (at 140.4621 58.2941 90)
-      (effects (font (size 1.27 1.27)) (justify left))
-    )
-    (property "Value" "15MQ040N" (id 1) (at 140.4621 60.5928 90)
-      (effects (font (size 1.27 1.27)) (justify left))
-    )
-    (property "Footprint" "Diode_SMD:D_SMA" (id 2) (at 138.43 59.055 0)
-      (effects (font (size 1.27 1.27)) hide)
-    )
-    (property "Datasheet" "~" (id 3) (at 138.43 59.055 0)
+  (symbol (lib_id "Device:D") (at 121.92 66.04 180) (unit 1)
+    (in_bom yes) (on_board yes) (fields_autoplaced)
+    (property "Reference" "D1" (id 0) (at 121.92 61.3368 0))
+    (property "Value" "15MQ040N" (id 1) (at 121.92 63.6355 0))
+    (property "Footprint" "Diode_SMD:D_SMA" (id 2) (at 121.92 66.04 0)
+      (effects (font (size 1.27 1.27)) hide)
+    )
+    (property "Datasheet" "~" (id 3) (at 121.92 66.04 0)
       (effects (font (size 1.27 1.27)) hide)
     )
@@
     (pin "2")
   )
-  (symbol (lib_id "Device:C") (at 125.73 71.12 0) (unit 1)
-    (in_bom yes) (on_board yes)
-    (property "Reference" "C4" (id 0) (at 128.6511 69.9706 0)
-      (effects (font (size 1.27 1.27)) (justify left))
-    )
-    (property "Value" "100nF" (id 1) (at 128.651 72.269 0)
-      (effects (font (size 1.27 1.27)) (justify left))
-    )
-    (property "Footprint" "Capacitor_SMD:C_0603_1608Metric" (id 2) (at 126.6952 74.93 0)
-      (effects (font (size 1.27 1.27)) hide)
-    )
-    (property "Datasheet" "~" (id 3) (at 125.73 71.12 0)
-      (effects (font (size 1.27 1.27)) hide)
-    )
-    (property "UST_ID" "5c70984712875079b91f8b4c" (id 4) (at 125.73 71.12 0)
+  (symbol (lib_id "Device:C") (at 128.905 71.12 0) (unit 1)
+    (in_bom yes) (on_board yes)
+    (property "Reference" "C4" (id 0) (at 131.8261 69.9706 0)
+      (effects (font (size 1.27 1.27)) (justify left))
+    )
+    (property "Value" "100nF" (id 1) (at 131.826 72.269 0)
+      (effects (font (size 1.27 1.27)) (justify left))
+    )
+    (property "Footprint" "Capacitor_SMD:C_0603_1608Metric" (id 2) (at 129.8702 74.93 0)
+      (effects (font (size 1.27 1.27)) hide)
+    )
+    (property "Datasheet" "~" (id 3) (at 128.905 71.12 0)
+      (effects (font (size 1.27 1.27)) hide)
+    )
+    (property "UST_ID" "5c70984712875079b91f8b4c" (id 4) (at 128.905 71.12 0)
       (effects (font (size 1.27 1.27)) hide)
     )
@@
       (reference "#PWR0117") (unit 1) (value "GND") (footprint "")
     )
+    (path "/8657520c-1e53-4d66-bc84-0c8cc37faf4b"
+      (reference "#PWR?") (unit 1) (value "+5V") (footprint "")
+    )
     (path "/851230d7-1bf4-4256-81a4-a4f9cc4bb316"

Commit message: Edit PCB
Other:
- note added: "to DEVICE"
- note added: "to FMU"
Changed lines of the file:
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@@
     (stroke (width 0) (type solid) (color 0 0 0 0))
+  )
+  (text "to DEVICE" (at 213.995 93.345 180)
+    (effects (font (size 1.524 1.524)) (justify right bottom))
+  )
+  (text "to FMU" (at 252.73 93.345 180)
+    (effects (font (size 1.524 1.524)) (justify right bottom))
   )
   (text "Budou tu LED?" (at 269.24 18.415 180)

Commit message: Edit SCH and PCB
Connections:
- net #CTS: now also J2.4; no longer J2.5
- net #RTS: now also J2.5; no longer J2.4
Changed lines of the file:
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@@
     (effects (font (size 1.524 1.524)) (justify left bottom))
   )
-  (label "#RTS" (at 193.04 104.14 0)
+  (label "#CTS" (at 193.04 104.14 0)
     (effects (font (size 1.524 1.524)) (justify left bottom))
   )
-  (label "#CTS" (at 193.04 106.68 0)
+  (label "#RTS" (at 193.04 106.68 0)
     (effects (font (size 1.524 1.524)) (justify left bottom))
   )

Commit message: Edit PCB
Parts:
- added D4: GREEN, LED_SMD:LED_0603_1608Metric, symbol Device:LED
- added R7: 270R, Resistor_SMD:R_0603_1608Metric, symbol Device:R
- D2, D3: footprint LED_SMD:LED_0603_1608Metric_Castellated -> LED_SMD:LED_0603_1608Metric
- F1: value Fuse -> 750mA
Connections:
- net +5V: now also D4.2 (A); no longer R3.1
- net GND: now also R7.2
- net VBUS: now also R3.1
- new net: D4.1 (K), R7.1
Other:
- moved on the sheet: C1, C3, D1, D2, D3, F1, FB1, M1, M2, M3, M4, M5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
