File: hw/sch_pcb/TFUSBSERIAL01.kicad_pcb (KiCad board)
At the start: 2 copper layers, 30 x 30 mm, 29 parts, among them J1 USBC_USB4105-GF-A, J2 SM06B-GHS-TB, J3 SM06B-GHS-TB, M1 HOLE_TF, M2 HOLE_TF, M3 HOLE_TF, M4 HOLE_TF, M5 HOLE_TF, M6 HOLE_TF, U1 USBLC6-2SC6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

Commit message: usb serial
Parts:
- added FID1: Fiducial, Fiducial:Fiducial_1mm_Mask2mm, B.Cu at (149.4, 108.6)
- added FID2: Fiducial, Fiducial:Fiducial_1mm_Mask2mm, B.Cu at (156.1, 91.6)
- added R10: 100R, Resistor_SMD:R_0603_1608Metric, B.Cu at (156.8, 102.1)
- added R11: 100R, Resistor_SMD:R_0603_1608Metric, B.Cu at (150.1, 105.1)
- added R8: 100R, Resistor_SMD:R_0603_1608Metric, B.Cu at (156.3, 96.5)
- added R9: 100R, Resistor_SMD:R_0603_1608Metric, B.Cu at (153.7, 106.2)
- added TP1: #DTR, TestPoint:TestPoint_Pad_D1.0mm, F.Cu at (153.6, 106.7)
- added TP2: #DSR, TestPoint:TestPoint_Pad_D1.0mm, F.Cu at (151.2, 106.7)
- added TP3: #DCD, TestPoint:TestPoint_Pad_D1.0mm, F.Cu at (151.2, 104.6)
- added TP4: #RI, TestPoint:TestPoint_Pad_D1.0mm, F.Cu at (153.6, 104.6)
- F1: value 750mA -> 350mA; footprint Mlab_F:1812 -> Fuse:Fuse_0805_2012Metric
- R5: value 270R -> 290R
- R6, R7: value 270R -> 140R
- moved R7 35.0 mm to (142.3, 112.0), turned to 90 degrees
- moved F1 24.2 mm to (155.4, 89.5), turned to 0 degrees
- moved D1 12.8 mm to (161.6, 100.3), turned to 0 degrees
- moved D4 10.6 mm to (140.6, 112.0), turned to 90 degrees
- moved C1 7.20 mm to (148.2, 105.0), turned to 90 degrees
- moved C3 4.79 mm to (144.8, 107.1), turned to 90 degrees
- moved FB1 3.17 mm to (146.5, 106.1), turned to -90 degrees
- moved C4 2.01 mm to (153.4, 95.9), turned to 90 degrees
- moved C5 1.56 mm to (155.3, 105.1), turned to -90 degrees
- moved U2 1.55 mm to (153.4, 100.7)
- moved U1 1.15 mm to (148.0, 100.3)
- moved C2 0.94 mm to (151.5, 96.5), turned to 90 degrees
- moved R3 0.44 mm to (151.6, 93.8)
- moved J2 0.42 mm to (162.4, 92.4)
- moved J3 0.38 mm to (162.4, 108.2)
Connections:
- C1 pad 1: Net-(C1-Pad1) -> /VBUS
- C3 pad 1: Net-(D1-A) -> +5V
- C5 pad 1: GND -> Net-(U2-3V3OUT)
- C5 pad 2: Net-(U2-3V3OUT) -> GND
- D1 pad 1: +5V -> Net-(D1-K)
- F1 pad 1: /VBUS -> +5V
- F1 pad 2: Net-(C1-Pad1) -> Net-(D1-A)
- FB1 pad 1: Net-(C1-Pad1) -> /VBUS
- FB1 pad 2: Net-(D1-A) -> +5V
- J2 pad 1: +5V -> Net-(D1-A)
- J3 pad 1: +5V -> Net-(D1-K)
- U2 pad 1: /RXD -> Net-(U2-RXD)
- U2 pad 17: /TXD -> Net-(U2-TXD)
- U2 pad 18: unconnected-(U2-~{DTR}-Pad18) -> Net-(U2-~{DTR})
- U2 pad 19: /#RTS -> Net-(U2-~{RTS})
- U2 pad 2: unconnected-(U2-~{RI}-Pad2) -> Net-(U2-~{RI})
- U2 pad 4: unconnected-(U2-~{DSR}-Pad4) -> Net-(U2-~{DSR})
- U2 pad 5: unconnected-(U2-~{DCD}-Pad5) -> Net-(U2-~{DCD})
- U2 pad 6: /#CTS -> Net-(U2-~{CTS})
Routing:
- net GND: track 10.8 -> 0.07 mm, vias 49 -> 33
- net Net-(U2-~{DTR}): track 0.00 -> 9.35 mm, vias 0 -> 1
- net +5V: track 64.9 -> 56.2 mm, vias 4 -> 2
- net Net-(D1-A): track 10.3 -> 16.6 mm, vias 0 -> 2
- net /#CTS: track 39.2 -> 33.1 mm
- net Net-(C1-Pad1): track 5.55 -> 0.00 mm
- net Net-(U2-3V3OUT): track 14.3 -> 9.35 mm
- net /#RTS: track 19.8 -> 24.7 mm
- net /VBUS: track 26.2 -> 21.5 mm
- net Net-(U2-~{DSR}): track 0.00 -> 4.38 mm, vias 0 -> 1
- net Net-(D1-K): track 0.00 -> 3.80 mm
- net Net-(U2-TXD): track 0.00 -> 3.59 mm
- net /RXD: track 25.5 -> 21.9 mm
- net Net-(U2-~{CTS}): track 0.00 -> 3.16 mm
- net Net-(U2-~{DCD}): track 0.00 -> 3.10 mm, vias 0 -> 1
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
Commit message: update silkscreen
Other:
- board text added: "to PERIP."
- board text added: "to PERIPHERAL"
- board text removed: "to DEVICE"
Changed lines of the file:
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@@
     (property "ki_keywords" "diode")
     (attr smd)
-    (fp_text reference "D1" (at -2.4 -2.2) (layer "B.SilkS")
+    (fp_text reference "D1" (at 2.8 -1.4) (layer "B.SilkS")
         (effects (font (size 0.8 0.8) (thickness 0.15)) (justify mirror))
     )
@@
     (effects (font (size 1 1) (thickness 0.2) bold) (justify bottom mirror))
   )
-  (gr_text "to DEVICE" (at 158.5 92.6 270) (layer "B.SilkS")
+  (gr_text "to PERIPHERAL" (at 158.3 92.6 270) (layer "B.SilkS")
     (effects (font (size 1 1) (thickness 0.2) bold) (justify mirror))
   )
@@
     (effects (font (size 1.5 1.5) (thickness 0.3)))
   )
-  (gr_text "to DEVICE" (at 163.8 92.9 90) (layer "F.SilkS")
+  (gr_text "to PERIP." (at 163.7 92.9 90) (layer "F.SilkS")
     (effects (font (size 1.5 1.5) (thickness 0.3)))
   )
