File: hw/sch_pcb/TFUSBSERIAL01.kicad_pcb (KiCad board)
At the start: 2 copper layers, 30 x 30 mm, 39 parts, among them J1 USBC_USB4105-GF-A, J2 SM06B-GHS-TB, J3 SM06B-GHS-TB, M1 HOLE_TF, M2 HOLE_TF, M3 HOLE_TF, M4 HOLE_TF, M5 HOLE_TF, M6 HOLE_TF, U1 USBLC6-2SC6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

Commit message: layout updates
Parts:
- FID1, FID2: footprint Fiducial:Fiducial_1mm_Mask2mm -> Fiducial:Fiducial_0.5mm_Mask1mm
- R5: value 290R -> 287R
- R6, R7: value 140R -> 130R
- moved C1 0.88 mm to (148.2, 105.9)
- moved R11 0.87 mm to (149.7, 105.9)
- moved C4 0.41 mm to (153.3, 96.3)
- moved C2 0.17 mm to (151.5, 96.3)
Routing:
- net Net-(U2-~{DCD}): track 3.10 -> 4.06 mm
- net Net-(U2-~{CTS}): track 3.16 -> 4.11 mm
- net /RXLED/CBUS1: track 10.7 -> 11.3 mm
- net Net-(U2-3V3OUT): track 9.35 -> 9.93 mm
- net Net-(J1-CC1): track 10.8 -> 11.3 mm
- net /VBUS: track 21.5 -> 22.0 mm
Other:
- rule pad_to_mask_clearance: 0.2 -> 0.1

Commit message: Kontrola a upravy pred vyrobou.
Parts:
- D1: value 15MQ040N -> SRL23; footprint Diode_SMD:D_SMA -> Diode_SMD:D_SOD-323_HandSoldering
Routing:
- net Net-(D1-A): track 16.6 -> 17.9 mm
- net Net-(D1-K): track 3.80 -> 4.74 mm
Other:
- rule pad_to_mask_clearance: 0.1 -> 0.2
Changed lines of the file:
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@@
       (dielectric_constraints no)
     )
-    (pad_to_mask_clearance 0.1)
+    (pad_to_mask_clearance 0.2)
     (pcbplotparams
       (layerselection 0x00010e0_ffffffff)
@@
       (net 32 "Net-(U2-~{DSR})") (pinfunction "1") (pintype "passive"))
   )
-  (footprint "Diode_SMD:D_SMA" (layer "B.Cu")
+  (footprint "Diode_SMD:D_SOD-323_HandSoldering" (layer "B.Cu")
     (at 161.6 100.3)
-    (descr "Diode SMA (DO-214AC)")
-    (tags "Diode SMA (DO-214AC)")
-    (property "Sheetfile" "TFUSBSERIAL01.kicad_sch")
-    (property "Sheetname" "")
-    (property "UST_ID" "5c70984512875079b91f88b0")
+    (descr "SOD-323")
+    (tags "SOD-323")
+    (property "Sheetfile" "TFUSBSERIAL01.kicad_sch")
+    (property "Sheetname" "")
+    (property "UST_ID" "")
     (property "ki_description" "Diode")
     (property "ki_keywords" "diode")
     (attr smd)
-    (fp_text reference "D1" (at 2.7 -1.6) (layer "B.SilkS")
-        (effects (font (size 0.8 0.8) (thickness 0.15)) (justify mirror))
-    )
-    (fp_text value "15MQ040N" (at 0 -2.6) (layer "B.Fab")
-        (effects (font (size 0.8 0.8) (thickness 0.15)) (justify mirror))
-    )
-    (fp_text user "${REFERENCE}" (at 0 2.5) (layer "B.Fab")
+    (fp_text reference "D1" (at -0.0052 1.6302 180) (layer "B.SilkS")
         (effects (font (size 1 1) (thickness 0.15)) (justify mirror))
     )
-    (fp_line (start -3.51 -1.65) (end 2 -1.65)
-      (stroke (width 0.12) (type solid)) (layer "B.SilkS"))
-    (fp_line (start -3.51 1.65) (end -3.51 -1.65)
-      (stroke (width 0.12) (type solid)) (layer "B.SilkS"))
-    (fp_line (start -3.51 1.65) (end 2 1.65)
-      (stroke (width 0.12) (type solid)) (layer "B.SilkS"))
-    (fp_line (start -3.5 -1.75) (end -3.5 1.75)
-      (stroke (width 0.05) (type solid)) (layer "B.CrtYd"))
-    (fp_line (start -3.5 1.75) (end 3.5 1.75)
-      (stroke (width 0.05) (type solid)) (layer "B.CrtYd"))
-    (fp_line (start 3.5 -1.75) (end -3.5 -1.75)
-      (stroke (width 0.05) (type solid)) (layer "B.CrtYd"))
-    (fp_line (start 3.5 1.75) (end 3.5 -1.75)
-      (stroke (width 0.05) (type solid)) (layer "B.CrtYd"))
-    (fp_line (start -2.3 -1.5) (end -2.3 1.5)
-      (stroke (width 0.1) (type solid)) (layer "B.Fab"))
-    (fp_line (start -0.64944 -0.00102) (end -1.55114 -0.00102)
-      (stroke (width 0.1) (type solid)) (layer "B.Fab"))
-    (fp_line (start -0.64944 -0.00102) (end 0.50118 -0.75032)
-      (stroke (width 0.1) (type solid)) (layer "B.Fab"))
-    (fp_line (start -0.64944 -0.00102) (end 0.50118 0.79908)
-      (stroke (width 0.1) (type solid)) (layer "B.Fab"))
-    (fp_line (start -0.64944 0.79908) (end -0.64944 -0.80112)
-      (stroke (width 0.1) (type solid)) (layer "B.Fab"))
-    (fp_line (start 0.50118 -0.75032) (end 0.50118 0.79908)
-      (stroke (width 0.1) (type solid)) (layer "B.Fab"))
-    (fp_line (start 0.50118 -0.00102) (end 1.4994 -0.00102)
-      (stroke (width 0.1) (type solid)) (layer "B.Fab"))
-    (fp_line (start 2.3 -1.5) (end -2.3 -1.5)
-      (stroke (width 0.1) (type solid)) (layer "B.Fab"))
-    (fp_line (start 2.3 1.5) (end -2.3 1.5)
-      (stroke (width 0.1) (type solid)) (layer "B.Fab"))
-    (fp_line (start 2.3 1.5) (end 2.3 -1.5)
-      (stroke (width 0.1) (type solid)) (layer "B.Fab"))
-    (pad "1" smd roundrect (at -2 0) (size 2.5 1.8) (layers "B.Cu" "B.Paste" "B.Mask") (roundrect_rratio 0.1388888889)
+    (fp_text value "SRL23" (at 0.1 -1.9 180) (layer "B.Fab")
+        (effects (font (size 1 1) (thickness 0.15)) (justify mirror))
+    )
+    (fp_text user "${REFERENCE}" (at 0 1.85 180) (layer "B.Fab")
+        (effects (font (size 1 1) (thickness 0.15)) (justify mirror))
+    )
+    (fp_line (start -2.01 -0.85) (end 1.25 -0.85)
+      (stroke (width 0.12) (type solid)) (layer "B.SilkS"))
+    (fp_line (start -2.01 0.85) (end -2.01 -0.85)
+      (stroke (width 0.12) (type solid)) (layer "B.SilkS"))
+    (fp_line (start -2.01 0.85) (end 1.25 0.85)
+      (stroke (width 0.12) (type solid)) (layer "B.SilkS"))
+    (fp_line (start -2 -0.95) (end 2 -0.95)
+      (stroke (width 0.05) (type solid)) (layer "B.CrtYd"))
+    (fp_line (start -2 0.95) (end -2 -0.95)
+      (stroke (width 0.05) (type solid)) (layer "B.CrtYd"))
+    (fp_line (start -2 0.95) (end 2 0.95)
+      (stroke (width 0.05) (type solid)) (layer "B.CrtYd"))
+    (fp_line (start 2 0.95) (end 2 -0.95)
+      (stroke (width 0.05) (type solid)) (layer "B.CrtYd"))
+    (fp_line (start -0.9 -0.7) (end -0.9 0.7)
+      (stroke (width 0.1) (type solid)) (layer "B.Fab"))
+    (fp_line (start -0.9 0.7) (end 0.9 0.7)
+      (stroke (width 0.1) (type solid)) (layer "B.Fab"))
+    (fp_line (start -0.3 0) (end -0.5 0)
+      (stroke (width 0.1) (type solid)) (layer "B.Fab"))
+    (fp_line (start -0.3 0) (end 0.2 0.35)
+      (stroke (width 0.1) (type solid)) (layer "B.Fab"))
+    (fp_line (start -0.3 0.35) (end -0.3 -0.35)
+      (stroke (width 0.1) (type solid)) (layer "B.Fab"))
+    (fp_line (start 0.2 -0.35) (end -0.3 0)
+      (stroke (width 0.1) (type solid)) (layer "B.Fab"))
+    (fp_line (start 0.2 0) (end 0.45 0)
+      (stroke (width 0.1) (type solid)) (layer "B.Fab"))
+    (fp_line (start 0.2 0.35) (end 0.2 -0.35)
+      (stroke (width 0.1) (type solid)) (layer "B.Fab"))
+    (fp_line (start 0.9 -0.7) (end -0.9 -0.7)
+      (stroke (width 0.1) (type solid)) (layer "B.Fab"))
+    (fp_line (start 0.9 0.7) (end 0.9 -0.7)
+      (stroke (width 0.1) (type solid)) (layer "B.Fab"))
+    (pad "1" smd roundrect (at -1.25 0) (size 1 1) (layers "B.Cu" "B.Paste" "B.Mask") (roundrect_rratio 0.25)
       (net 2 "Net-(D1-K)") (pinfunction "K") (pintype "passive"))
-    (pad "2" smd roundrect (at 2 0) (size 2.5 1.8) (layers "B.Cu" "B.Paste" "B.Mask") (roundrect_rratio 0.1388888889)
+    (pad "2" smd roundrect (at 1.25 0) (size 1 1) (layers "B.Cu" "B.Paste" "B.Mask") (roundrect_rratio 0.25)
       (net 4 "Net-(D1-A)") (pinfunction "A") (pintype "passive"))
-    (model "${KICAD6_3DMODEL_DIR}/Diode_SMD.3dshapes/D_SMA.wrl"
+    (model "${KICAD6_3DMODEL_DIR}/Diode_SMD.3dshapes/D_SOD-323.wrl"
       (offset (xyz 0 0 0))
       (scale (xyz 1 1 1))
@@
   (via (at 148.441809 97.259855) (size 0.8) (drill 0.4) (layers "F.Cu" "B.Cu") (free) (net 1))
   (via (at 156 86.8) (size 0.8) (drill 0.4) (layers "F.Cu" "B.Cu") (free) (net 1))
-  (via (at 155.1 111.4) (size 0.8) (drill 0.4) (layers "F.Cu" "B.Cu") (free) (net 1))
+  (via (at 155.1 110.9472) (size 0.8) (drill 0.4) (layers "F.Cu" "B.Cu") (free) (net 1))
   (via (at 145.119 104.141) (size 0.8) (drill 0.4) (layers "F.Cu" "B.Cu") (free) (net 1))
   (via (at 146.2 90.4) (size 0.8) (drill 0.4) (layers "F.Cu" "B.Cu") (free) (net 1))
@@
   (via (at 147.4 95.7) (size 0.8) (drill 0.4) (layers "F.Cu" "B.Cu") (free) (net 1))
   (segment (start 152.9605 101.317) (end 152.9605 101.3895) (width 0.2) (layer "B.Cu") (net 1))
+  (segment (start 160.6 104.858) (end 160.6 100.55) (width 0.4) (layer "B.Cu") (net 2))
   (segment (start 160.6 105.016) (end 160.541 105.075) (width 0.5) (layer "B.Cu") (net 2))
-  (segment (start 160.6 101.142) (end 160.6 104.858) (width 0.4) (layer "B.Cu") (net 2))
+  (segment (start 160.6 100.55) (end 160.35 100.3) (width 0.4) (layer "B.Cu") (net 2))
   (segment (start 151.4 99.2) (end 155 102.8) (width 0.3) (layer "F.Cu") (net 3))
   (segment (start 155 102.8) (end 155.1495 102.8) (width 0.3) (layer "F.Cu") (net 3))
@@
   (via (at 162.255 89.4) (size 0.8) (drill 0.4) (layers "F.Cu" "B.Cu") (net 4))
   (via (at 163.7 99.4) (size 0.8) (drill 0.4) (layers "F.Cu" "B.Cu") (net 4))
+  (segment (start 162.85 100.25) (end 163.7 99.4) (width 0.5) (layer "B.Cu") (net 4))
   (segment (start 162.255 89.4) (end 156.4 89.4) (width 0.3) (layer "B.Cu") (net 4))
+  (segment (start 162.85 100.3) (end 162.85 100.25) (width 0.5) (layer "B.Cu") (net 4))
   (segment (start 156.4 89.4) (end 156.3 89.5) (width 0.3) (layer "B.Cu") (net 4))
   (segment (start 146.35994 100.300014) (end 146.5 100.159954) (width 0.4) (layer "F.Cu") (net 5))

Commit message: Aisler custom bridges
Other:
- board size 30 x 30 mm -> 30 x 36 mm
Changed lines of the file:
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@@
     (comment 2 "Short description\\nTwo lines are maximum")
     (comment 3 "nickname <email@example.com>")
+    (comment 4 "AISLER Project ID: JJMRKJQJ")
   )
   (layers
@@
     (fp_line (start 2 2) (end 2 -2)
       (stroke (width 0.1) (type solid)) (layer "B.Fab"))
-    (pad "" smd roundrect (at -0.625 -0.625 90) (size 1.01 1.01) (layers "B.Paste") (roundrect_rratio 0.247525))
-    (pad "" smd roundrect (at -0.625 0.625 90) (size 1.01 1.01) (layers "B.Paste") (roundrect_rratio 0.247525))
-    (pad "" smd roundrect (at 0.625 -0.625 90) (size 1.01 1.01) (layers "B.Paste") (roundrect_rratio 0.247525))
-    (pad "" smd roundrect (at 0.625 0.625 90) (size 1.01 1.01) (layers "B.Paste") (roundrect_rratio 0.247525))
+    (pad "" smd roundrect (at -0.625 -0.625 90) (size 1.01 1.01) (layers "B.Paste") (roundrect_rratio 0.2475247525))
+    (pad "" smd roundrect (at -0.625 0.625 90) (size 1.01 1.01) (layers "B.Paste") (roundrect_rratio 0.2475247525))
+    (pad "" smd roundrect (at 0.625 -0.625 90) (size 1.01 1.01) (layers "B.Paste") (roundrect_rratio 0.2475247525))
+    (pad "" smd roundrect (at 0.625 0.625 90) (size 1.01 1.01) (layers "B.Paste") (roundrect_rratio 0.2475247525))
     (pad "1" smd roundrect (at -1.9375 1 90) (size 0.825 0.25) (layers "B.Cu" "B.Paste" "B.Mask") (roundrect_rratio 0.25)
       (net 24 "Net-(U2-RXD)") (pinfunction "RXD") (pintype "input"))
@@
     )
     (stroke (width 0) (type solid)) (fill solid) (layer "F.SilkS"))
+  (gr_line (start 162 85.3) (end 162 82.3)
+    (stroke (width 0.05588) (type default)) (layer "Edge.Cuts"))
   (gr_line (start 135.594 85.317) (end 135.594 115.317)
     (stroke (width 0.15) (type solid)) (layer "Edge.Cuts"))
@@
   (gr_line (start 135.594 115.317) (end 165.594 115.317)
     (stroke (width 0.15) (type solid)) (layer "Edge.Cuts"))
+  (gr_line (start 162 118.3) (end 162 115.3)
+    (stroke (width 0.05588) (type default)) (layer "Edge.Cuts"))
+  (gr_line (start 142 118.3) (end 142 115.3)
+    (stroke (width 0.05588) (type default)) (layer "Edge.Cuts"))
   (gr_line (start 165.594 85.317) (end 135.594 85.317)
     (stroke (width 0.15) (type solid)) (layer "Edge.Cuts"))
+  (gr_line (start 142 85.3) (end 142 82.3)
+    (stroke (width 0.05588) (type default)) (layer "Edge.Cuts"))
   (gr_text "TFUSBSERIAL01A\n" (at 151.2 113.3) (layer "B.Cu")
     (effects (font (size 1 1) (thickness 0.2) bold) (justify bottom mirror))
