File: hw/sch_pcb/TFUSBSERIAL01.kicad_pcb (KiCad board)
At the start: 2 copper layers, 30 x 30 mm, 39 parts, among them J1 USBC_USB4105-GF-A, J2 SM06B-GHS-TB, J3 SM06B-GHS-TB, M1 HOLE_TF, M2 HOLE_TF, M3 HOLE_TF, M4 HOLE_TF, M5 HOLE_TF, M6 HOLE_TF, U1 USBLC6-2SC6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

Commit message: Fixing #4 WIP.
Parts:
- added JP1: SolderJumper_3_Bridged12, Jumper:SolderJumper-3_P1.3mm_Bridged12_Pad1.0x1.5mm_NumberLabels, F.Cu at (156.2, 109.7)
Connections:
- net Net-(U2-~{DTR}) renamed /#DTR
- J2 pad 5: /#RTS -> Net-(JP1-C)
Other:
- board text added: "2026"
- board text added: "TFUSBSERIAL01B"
- board text removed: "2023"
- board text removed: "TFUSBSERIAL01A"
