File: hw/sch_pcb/TFUSBSERIAL01.kicad_sch (KiCad schematic)
At the start: 39 parts, among them J1 USBC_USB4105-GF-A, J2 SM06B-GHS-TB, J3 SM06B-GHS-TB, M1 HOLE_TF, M2 HOLE_TF, M3 HOLE_TF, M4 HOLE_TF, M5 HOLE_TF, M6 HOLE_TF, U1 USBLC6-2SC6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

Commit message: exclude mechanical components from BOM.
Parts:
- FID2, M1, M2, M3, M4, M5, M6, TP1, TP2, TP3, TP4: now left out of the parts list
Changed lines of the file:
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@@
   )
   (symbol (lib_id "MLAB_MECHANICAL:HOLE_TF") (at 243.205 16.51 0) (unit 1)
-    (in_bom yes) (on_board yes) (dnp no) (fields_autoplaced)
+    (in_bom no) (on_board yes) (dnp no) (fields_autoplaced)
     (property "Reference" "M1" (at 244.6021 15.6224 0)
       (effects (font (size 1.524 1.524)) (justify left))
@@
     (property "Datasheet" "" (at 243.205 16.51 0)
       (effects (font (size 1.524 1.524)))
+    )
+    (property "Sim.Enable" "0" (at 243.205 16.51 0)
+      (effects (font (size 1.27 1.27)) hide)
     )
     (instances
@@
   )
   (symbol (lib_id "Connector:TestPoint") (at 172.72 111.76 270) (unit 1)
-    (in_bom yes) (on_board yes) (dnp no)
+    (in_bom no) (on_board yes) (dnp no)
     (property "Reference" "TP4" (at 177.419 110.736 90)
       (effects (font (size 1.27 1.27)) (justify left))
@@
     )
     (property "Datasheet" "~" (at 172.72 116.84 0)
+      (effects (font (size 1.27 1.27)) hide)
+    )
+    (property "Sim.Enable" "0" (at 172.72 111.76 0)
       (effects (font (size 1.27 1.27)) hide)
     )
@@
   )
   (symbol (lib_id "Connector:TestPoint") (at 172.72 109.22 270) (unit 1)
-    (in_bom yes) (on_board yes) (dnp no)
+    (in_bom no) (on_board yes) (dnp no)
     (property "Reference" "TP3" (at 177.419 108.196 90)
       (effects (font (size 1.27 1.27)) (justify left))
@@
       (effects (font (size 1.27 1.27)) hide)
     )
+    (property "Sim.Enable" "0" (at 172.72 109.22 0)
+      (effects (font (size 1.27 1.27)) hide)
+    )
     (pin "1")
     (instances
@@
   )
   (symbol (lib_id "MLAB_MECHANICAL:HOLE_TF") (at 257.175 16.51 0) (unit 1)
-    (in_bom yes) (on_board yes) (dnp no) (fields_autoplaced)
+    (in_bom no) (on_board yes) (dnp no) (fields_autoplaced)
     (property "Reference" "M3" (at 258.5721 15.6224 0)
       (effects (font (size 1.524 1.524)) (justify left))
@@
     (property "Datasheet" "" (at 257.175 16.51 0)
       (effects (font (size 1.524 1.524)))
+    )
+    (property "Sim.Enable" "0" (at 257.175 16.51 0)
+      (effects (font (size 1.27 1.27)) hide)
     )
     (instances
@@
   )
   (symbol (lib_id "MLAB_MECHANICAL:HOLE_TF") (at 257.175 22.86 0) (unit 1)
-    (in_bom yes) (on_board yes) (dnp no) (fields_autoplaced)
+    (in_bom no) (on_board yes) (dnp no) (fields_autoplaced)
     (property "Reference" "M4" (at 258.5721 21.9724 0)
       (effects (font (size 1.524 1.524)) (justify left))
@@
     (property "Datasheet" "" (at 257.175 22.86 0)
       (effects (font (size 1.524 1.524)))
+    )
+    (property "Sim.Enable" "0" (at 257.175 22.86 0)
+      (effects (font (size 1.27 1.27)) hide)
     )
     (instances
@@
   )
   (symbol (lib_id "Connector:TestPoint") (at 172.72 104.14 270) (unit 1)
-    (in_bom yes) (on_board yes) (dnp no)
+    (in_bom no) (on_board yes) (dnp no)
     (property "Reference" "TP1" (at 177.419 103.116 90)
       (effects (font (size 1.27 1.27)) (justify left))
@@
       (effects (font (size 1.27 1.27)) hide)
     )
+    (property "Sim.Enable" "0" (at 172.72 104.14 0)
+      (effects (font (size 1.27 1.27)) hide)
+    )
     (pin "1")
     (instances
@@
   )
   (symbol (lib_id "MLAB_MECHANICAL:HOLE_TF") (at 269.875 22.86 0) (unit 1)
-    (in_bom yes) (on_board yes) (dnp no) (fields_autoplaced)
+    (in_bom no) (on_board yes) (dnp no) (fields_autoplaced)
     (property "Reference" "M6" (at 271.2721 21.9724 0)
       (effects (font (size 1.524 1.524)) (justify left))
@@
       (effects (font (size 1.524 1.524)))
     )
+    (property "Sim.Enable" "0" (at 269.875 22.86 0)
+      (effects (font (size 1.27 1.27)) hide)
+    )
     (instances
       (project "TFUSBSERIAL01"
@@
   )
   (symbol (lib_id "MLAB_MECHANICAL:HOLE_TF") (at 243.205 22.86 0) (unit 1)
-    (in_bom yes) (on_board yes) (dnp no) (fields_autoplaced)
+    (in_bom no) (on_board yes) (dnp no) (fields_autoplaced)
     (property "Reference" "M2" (at 244.6021 21.9724 0)
       (effects (font (size 1.524 1.524)) (justify left))
@@
     (property "Datasheet" "" (at 243.205 22.86 0)
       (effects (font (size 1.524 1.524)))
+    )
+    (property "Sim.Enable" "0" (at 243.205 22.86 0)
+      (effects (font (size 1.27 1.27)) hide)
     )
     (instances
@@
   )
   (symbol (lib_id "Connector:TestPoint") (at 172.72 106.68 270) (unit 1)
-    (in_bom yes) (on_board yes) (dnp no)
+    (in_bom no) (on_board yes) (dnp no)
     (property "Reference" "TP2" (at 177.419 105.656 90)
       (effects (font (size 1.27 1.27)) (justify left))
@@
     )
     (property "Datasheet" "~" (at 172.72 111.76 0)
+      (effects (font (size 1.27 1.27)) hide)
+    )
+    (property "Sim.Enable" "0" (at 172.72 106.68 0)
       (effects (font (size 1.27 1.27)) hide)
     )
@@
   )
   (symbol (lib_id "MLAB_MECHANICAL:HOLE_TF") (at 269.875 16.51 0) (unit 1)
-    (in_bom yes) (on_board yes) (dnp no) (fields_autoplaced)
+    (in_bom no) (on_board yes) (dnp no) (fields_autoplaced)
     (property "Reference" "M5" (at 271.2721 15.6224 0)
       (effects (font (size 1.524 1.524)) (justify left))
@@
     (property "Datasheet" "" (at 269.875 16.51 0)
       (effects (font (size 1.524 1.524)))
+    )
+    (property "Sim.Enable" "0" (at 269.875 16.51 0)
+      (effects (font (size 1.27 1.27)) hide)
     )
     (instances
@@
       (effects (font (size 1.27 1.27)) hide)
     )
-    (property "Datasheet" "~" (at 247.65 118.11 0)
+    (property "Datasheet" "https://www.tme.eu/Document/039d7772a3e1de850ecf12d397e62c7b/srl23.pdf" (at 247.65 118.11 0)
       (effects (font (size 1.27 1.27)) hide)
     )
@@
   )
   (symbol (lib_id "Mechanical:Fiducial") (at 227.33 22.86 0) (unit 1)
-    (in_bom yes) (on_board yes) (dnp no) (fields_autoplaced)
+    (in_bom no) (on_board yes) (dnp no) (fields_autoplaced)
     (property "Reference" "FID2" (at 229.87 21.59 0)
       (effects (font (size 1.27 1.27)) (justify left))
@@
       (effects (font (size 1.27 1.27)) hide)
     )
+    (property "Sim.Enable" "0" (at 227.33 22.86 0)
+      (effects (font (size 1.27 1.27)) hide)
+    )

Commit message: Edit UST_ID
Parts:
- R5: UST_ID 5c70984512875079b91f8969 -> 651a975c462c6d9e7205504d
Changed lines of the file:
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@@
       (effects (font (size 1.27 1.27)) hide)
     )
-    (property "UST_ID" "5c70984512875079b91f8969" (at 260.35 61.595 0)
+    (property "UST_ID" "651a975c462c6d9e7205504d" (at 260.35 61.595 0)
       (effects (font (size 1.27 1.27)) hide)
     )
