File: hw/sch_pcb/TFUSBSERIAL01.kicad_sch (KiCad schematic)
At the start: 39 parts, among them J1 USBC_USB4105-GF-A, J2 SM06B-GHS-TB, J3 SM06B-GHS-TB, M1 HOLE_TF, M2 HOLE_TF, M3 HOLE_TF, M4 HOLE_TF, M5 HOLE_TF, M6 HOLE_TF, U1 USBLC6-2SC6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

Commit message: Fixing #4 WIP.
Parts:
- added JP1: SolderJumper_3_Bridged12, Jumper:SolderJumper-3_P1.3mm_Bridged12_Pad1.0x1.5mm_NumberLabels, symbol Jumper:SolderJumper_3_Bridged12
Connections:
- net #RTS: now also JP1.3 (B); no longer J2.5
- net #DTR: now reaches TP1.1, U2.18 (~{DTR})
- net #DTR: now also JP1.1 (A)
- new net: J2.5, JP1.2 (C)
Other:
- title: TFUSBSERIAL01A -> TFUSBSERIAL01B
- moved on the sheet: C1, C3, C4, D2, D3, D4, FB1, J2, J3, R10, R11, R5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
